File: CRAB_flipdot.kicad_pcb (KiCad board)
At the start: 2 copper layers, 65 x 56 mm, 27 parts, among them J1 Screw_Terminal_01x04, J2 Conn_01x03, J3 RJ11, Q1 Q_NMOS_DGS, U1 R-785.0-1.0, U2 sn65hvd72d

Commit message: Prototype ready
Parts:
- added R8: 100R, Resistors_SMD:R_0805_HandSoldering, F.Cu at (192.4, 75.6)
- C1: footprint Capacitors_SMD:CP_Elec_4x4.5 -> Capacitors_SMD:CP_Elec_6.3x4.5
- Q1: value Q_NMOS_DGS -> Q_NMOS_GDS; footprint TO_SOT_Packages_SMD:SOT-23 -> TO_SOT_Packages_SMD:SOT-23_Handsoldering
- moved Q1 8.82 mm to (200.0, 80.6), turned to 90 degrees
- moved U2 0.76 mm to (183.4, 72.4)
- moved R7 0.64 mm to (184.4, 87.0)
- moved C1 0.51 mm to (151.9, 81.9)
Connections:
- Q1 pad 2: Net-(H1-Pad8) -> Net-(Q1-Pad2)
- R3 pad 2: Net-(Q1-Pad1) -> Net-(Q1-Pad2)
Routing:
- net Net-(Q1-Pad2): track 0.00 -> 8.74 mm
- net Net-(H1-Pad8): track 55.3 -> 61.1 mm
- net +5V: track 115.2 -> 119.0 mm
- net Net-(Q1-Pad1): track 5.47 -> 8.81 mm
- net GND: track 79.3 -> 76.5 mm, vias 7 -> 6
- net Net-(D1-Pad2): track 44.5 -> 41.9 mm
- net A_OUT: track 59.8 -> 57.4 mm
- net Net-(R5-Pad2): track 12.1 -> 11.3 mm
- net Net-(R6-Pad2): track 8.57 -> 7.85 mm
- net B_OUT: track 50.1 -> 50.7 mm
Other:
- net class Default: trace_width 0.25 -> 0.33
